Commit message: third update

File: src/drone_ros2/sjtu_drone_description/urdf/sjtu_drone.urdf (robot description, URDF)
Before this commit: robot sjtu_drone, 5 links, 4 joints
Joints:
- joint bottom_cam_joint: origin xyz=0 0 0 rpy=0 1.570796326795 0 -> xyz=0 0 0 rpy=0 ${M_PI/2} 0
- joint sonar_joint: origin xyz=0 0 0 rpy=0 1.570796326795 0 -> xyz=0 0 0 rpy=0 ${M_PI/2} 0

File: src/drone_ros2/sjtu_drone_description/urdf/sjtu_drone.urdf.xacro (robot description, xacro)
@@ -57,13 +57,5 @@
     <plugin name='simple_drone' filename='libplugin_drone.so'>
       <ros>
-        <namespace>${mp['namespace']}</namespace>
         <remapping>cmd_vel:=cmd_vel</remapping>
-        <remapping>imu:=imu</remapping>
-        <remapping>sonar:=sonar</remapping>
-        <remapping>camera_front:=camera_front</remapping>
-        <remapping>camera_bottom:=camera_bottom</remapping>
-        <remapping>camera_front_info:=camera_front_info</remapping>
-        <remapping>camera_bottom_info:=camera_bottom_info</remapping>
-        <remapping>gps:=gps</remapping>
       </ros>
       <bodyName>base_link</bodyName>
@@ -119,9 +111,9 @@
       <plugin name='imu' filename='libgazebo_ros_imu_sensor.so'>
         <ros>
-          <namespace>${mp['namespace']}</namespace>
-          <!-- <remapping>imu:=imu</remapping> -->
+          <!-- <namespace>${mp['namespace']}</namespace> -->
+          <remapping>imu:=imu</remapping>
         </ros>
         <initial_orientation_as_reference>false</initial_orientation_as_reference>
-        <frame_name>${mp['namespace']}/base_link</frame_name>
+        <!-- <frame_name>${mp['namespace']}/base_link</frame_name> -->
       </plugin>
     </sensor>
@@ -161,44 +153,10 @@
       <plugin name="sonar" filename="libgazebo_ros_ray_sensor.so">
         <ros>
-          <namespace>${mp['namespace']}</namespace>
-          <!-- <remapping>~/out:=sonar</remapping> -->
-        </ros>
-        <frame_name>${mp['namespace']}/sonar_link</frame_name>
-        <output_type>sensor_msgs/Range</output_type>
-        <radiation_type>ultrasound</radiation_type>
-      </plugin>
-    </sensor>
-  </gazebo>
-  <gazebo reference="front_cam_link">
-    <sensor name="front_camera" type="camera">
-      <always_on>1</always_on>
-      <visualize>1</visualize>
-      <update_rate>60</update_rate>
-      <camera>
-        <horizontal_fov>2.09</horizontal_fov>
-        <image>
-          <width>640</width>
-          <height>360</height>
-          <format>R8G8B8</format>
-        </image>
-        <clip>
-          <near>0.1</near>
-          <far>100</far>
-        </clip>
-        <noise>
-          <type>gaussian</type>
-          <mean>0.0</mean>
-          <stddev>0.01</stddev>
-        </noise>
-      </camera>
-      <plugin name="camera_front" filename="libgazebo_ros_camera.so">
-        <ros>
-          <namespace>${mp['namespace']}</namespace>
-          <!-- <remapping>~/image_raw:=camera_front</remapping>
-          <remapping>~/camera_info:=camera_front_info</remapping> -->
-        </ros>
-        <frame_name>${mp['namespace']}/front_cam_link</frame_name>
-        <camera_name>front</camera_name>
-        <hack_baseline>0.07</hack_baseline>
+          <!-- <namespace>${mp['namespace']}</namespace> -->
+          <remapping>~/out:=sonar</remapping>
+        </ros>
+        <!-- <frame_name>${mp['namespace']}/sonar_link</frame_name> -->
+        <output_type>sensor_msgs/LaserScan</output_type>
+        <!-- <radiation_type>ultrasound</radiation_type> -->
       </plugin>
     </sensor>
@@ -206,5 +164,5 @@
   <!-- forward looking depth camera -->
   <gazebo reference="front_cam_link">
-    <sensor name="front_depth_camera" type="depth">
+    <sensor name="front_camera" type="depth">
       <always_on>1</always_on>
       <visualize>1</visualize>
@@ -222,49 +180,12 @@
         </clip>
       </camera>
-      <plugin filename="libgazebo_ros_camera.so" name="depth_camera_front">
-        <ros>
-          <namespace>/simple_drone</namespace>
+      <plugin name="camera_front" filename="libgazebo_ros_camera.so">
+        <!-- <ros> -->
+          <!-- <namespace>${mp['namespace']}e</namespace> -->
           <!-- <remapping>image_raw:=depth_camera_front</remapping>
           <remapping>camera_info:=depth_camera_front_info</remapping> -->
-        </ros>
-        <frame_name>/simple_drone/front_cam_link</frame_name>
-        <camera_name>depth_front</camera_name>
-        <min_depth>0.1</min_depth>
-        <max_depth>100.0</max_depth>
-      </plugin>
-    </sensor>
-  </gazebo>
-  <!-- downward looking camera -->
-  <gazebo reference="bottom_cam_link">
-    <sensor name="down_camera" type="camera">
-      <always_on>1</always_on>
-      <visualize>1</visualize>
-      <update_rate>15</update_rate>
-      <camera>
-        <horizontal_fov>1.047</horizontal_fov>
-        <image>
-          <width>640</width>
-          <height>360</height>
-          <format>R8G8B8</format>
-        </image>
-        <clip>
-          <near>0.1</near>
-          <far>100</far>
-        </clip>
-        <noise>
-          <type>gaussian</type>
-          <mean>0.0</mean>
-          <stddev>0.01</stddev>
-        </noise>
-      </camera>
-      <plugin name="camera_bottom" filename="libgazebo_ros_camera.so">
-        <ros>
-          <namespace>${mp['namespace']}</namespace>
-          <!-- <remapping>image_raw:=camera_bottom</remapping>
-          <remapping>camera_info:=camera_bottom_info</remapping> -->
-        </ros>
-        <frame_name>${mp['namespace']}/bottom_cam_link</frame_name>
-        <camera_name>bottom</camera_name>
-        <hack_baseline>0.07</hack_baseline>
+        <!-- </ros> -->
+        <frame_name>front_cam_link</frame_name>
+        <!-- <camera_name>front</camera_name> -->
       </plugin>
     </sensor>
@@ -272,5 +193,5 @@
   <!-- downward looking depth camera -->
   <gazebo reference="bottom_cam_link">
-    <sensor name="down_depth_camera" type="depth">
+    <sensor name="down_camera" type="depth">
       <always_on>1</always_on>
       <visualize>1</visualize>
@@ -288,14 +209,14 @@
         </clip>
       </camera>
-      <plugin filename="libgazebo_ros_camera.so" name="depth_camera_bottom">
-        <ros>
-          <namespace>/simple_drone</namespace>
+      <plugin name="camera_bottom" filename="libgazebo_ros_camera.so">
+        <!-- <ros> -->
+          <!-- <namespace>${mp['namespace']}</namespace> -->
           <!-- <remapping>image_raw:=depth_camera_bottom</remapping>
           <remapping>camera_info:=depth_camera_bottom_info</remapping> -->
-        </ros>
-        <frame_name>/simple_drone/bottom_cam_link</frame_name>
-        <camera_name>depth_bottom</camera_name>
-        <min_depth>0.1</min_depth>
-        <max_depth>100.0</max_depth>
+        <!-- </ros> -->
+        <frame_name>bottom_cam_link</frame_name>
+        <!-- <camera_name>bottom</camera_name> -->
+        <!-- <min_depth>0.1</min_depth> -->
+        <!-- <max_depth>100.0</max_depth> -->
       </plugin>
     </sensor>
@@ -304,5 +225,5 @@
     <sensor name="gps" type="gps">
       <always_on>1</always_on>
-      <update_rate>30</update_rate>
+      <update_rate>15</update_rate>
       <gps>
         <position_sensing>
@@ -323,8 +244,8 @@
       <plugin name="gps" filename="libgazebo_ros_gps_sensor.so">
         <ros>
-          <namespace>${mp['namespace']}</namespace>
+          <!-- <namespace>${mp['namespace']}</namespace> -->
           <remapping>~/out:=~/nav</remapping>
         </ros>
-        <frame_name>${mp['namespace']}/base_link</frame_name>
+        <!-- <frame_name>${mp['namespace']}/base_link</frame_name> -->
       </plugin>
     </sensor>
@@ -339,8 +260,8 @@
       <plugin name="collision_plugin" filename="libgazebo_ros_bumper.so">
         <ros>
-          <namespace>${mp['namespace']}</namespace>
-          <!-- <remapping>bumper_states:=bumper_states</remapping> -->
-        </ros>
-        <frame_name>${mp['namespace']}/base_link</frame_name>
+          <!-- <namespace>${mp['namespace']}</namespace> -->
+          <remapping>bumper_states:=bumper_states</remapping>
+        </ros>
+        <!-- <frame_name>${mp['namespace']}/base_link</frame_name> -->
       </plugin>
     </sensor>
